Commit message: Mujoco feature tested

File: crisp_ur_demos/config/ur.ros2_control.xacro (robot description, xacro)
@@ -1,10 +1,10 @@
 <?xml version="1.0"?>
 <robot xmlns:xacro="http://www.ros.org/wiki/xacro">
+  <!-- Keep these includes: they exist in the original file -->
   <xacro:include filename="$(find ur_description)/urdf/inc/ur_joint_control.xacro" />
   <xacro:include filename="$(find ur_description)/urdf/inc/ur_sensors.xacro" />
   <!--
-    Added 'mujoco_model' and 'ur_type' parameters.
-    - mujoco_model: path to the MuJoCo scene.xml (empty by default)
-    - ur_type: robot type (used to enable mujoco only for ur10e)
+    This macro name MUST remain "ur_ros2_control"
+    because ur.urdf.xacro calls <xacro:ur_ros2_control ... />
   -->
   <xacro:macro name="ur_ros2_control" params="
@@ -17,5 +17,6 @@
     output_recipe_filename
     transmission_hw_interface:=hardware_interface/PositionJointInterface
-    use_mock_hardware:=false mock_sensor_commands:=false
+    use_mock_hardware:=false
+    mock_sensor_commands:=false
     headless_mode:=false
     initial_positions:=${dict(shoulder_pan_joint=0.0,shoulder_lift_joint=-1.57,elbow_joint=0.0,wrist_1_joint=-1.57,wrist_2_joint=0.0,wrist_3_joint=0.0)}
@@ -30,26 +31,87 @@
     non_blocking_read:=true
     robot_receive_timeout:=0.04
-    mujoco_model:=
-    ur_type:=ur10e
+    mujoco_model:=''
     ">
+    <!-- Needed by the real driver (hash param), harmless for MuJoCo -->
     <xacro:property name="config_kinematics_parameters" value="${xacro.load_yaml(kinematics_parameters_file)}"/>
     <xacro:property name="sec_kinematics" value="${config_kinematics_parameters['kinematics']}" />
     <xacro:property name="kinematics_hash" value="${sec_kinematics['hash']}" scope="parent"/>
-    <!-- Add URDF transmission elements (for ros_control) -->
-    <!--<xacro:ur_arm_transmission prefix="${prefix}" hw_interface="${transmission_hw_interface}" />-->
-    <!-- Placeholder for ros2_control transmission which don't yet exist -->
+    <!-- IMPORTANT:
+         We cannot set mujoco_model default in params using $(find ...)
+         because xacro tries to parse it as an expression.
+         So we resolve it here. -->
     <ros2_control name="${name}" type="system">
-      <hardware>
-        <!-- Mock / simulator branch -->
-        <xacro:if value="${use_mock_hardware}">
-          <!-- Only enable mujoco simulator when:
-               - a mujoco_model path is provided, AND
-               - ur_type is 'ur10e' (we only have ur10e.xml) -->
-            <!-- Use the crisp_mujoco_sim simulator plugin (replace if your plugin name differs) -->
+      <!-- ========================================================= -->
+      <!-- A) MuJoCo mode (use_mock_hardware:=true) -->
+      <!-- ========================================================= -->
+      <xacro:if value="${use_mock_hardware}">
+        <hardware>
           <plugin>crisp_mujoco_sim/Simulator</plugin>
           <param name="mujoco_model">$(find crisp_ur_demos)/config/scene.xml</param>
-        </xacro:if>
-        <!-- Real-hardware branch -->
-        <xacro:unless value="${use_mock_hardware}">
+        </hardware>
+        <!-- IMPORTANT:
+             crisp_mujoco_sim/Simulator exports ONLY:
+               - effort command interface
+               - position/velocity/effort state interfaces
+             so we must declare ONLY those here
+        -->
+        <joint name="${tf_prefix}shoulder_pan_joint">
+          <command_interface name="effort"/>
+          <state_interface name="position">
+            <param name="initial_value">${initial_positions['shoulder_pan_joint']}</param>
+          </state_interface>
+          <state_interface name="velocity"/>
+          <state_interface name="effort"/>
+        </joint>
+        <joint name="${tf_prefix}shoulder_lift_joint">
+          <command_interface name="effort"/>
+          <state_interface name="position">
+            <param name="initial_value">${initial_positions['shoulder_lift_joint']}</param>
+          </state_interface>
+          <state_interface name="velocity"/>
+          <state_interface name="effort"/>
+        </joint>
+        <joint name="${tf_prefix}elbow_joint">
+          <command_interface name="effort"/>
+          <state_interface name="position">
+            <param name="initial_value">${initial_positions['elbow_joint']}</param>
+          </state_interface>
+          <state_interface name="velocity"/>
+          <state_interface name="effort"/>
+        </joint>
+        <joint name="${tf_prefix}wrist_1_joint">
+          <command_interface name="effort"/>
+          <state_interface name="position">
+            <param name="initial_value">${initial_positions['wrist_1_joint']}</param>
+          </state_interface>
+          <state_interface name="velocity"/>
+          <state_interface name="effort"/>
+        </joint>
+        <joint name="${tf_prefix}wrist_2_joint">
+          <command_interface name="effort"/>
+          <state_interface name="position">
+            <param name="initial_value">${initial_positions['wrist_2_joint']}</param>
+          </state_interface>
+          <state_interface name="velocity"/>
+          <state_interface name="effort"/>
+        </joint>
+        <joint name="${tf_prefix}wrist_3_joint">
+          <command_interface name="effort"/>
+          <state_interface name="position">
+            <param name="initial_value">${initial_positions['wrist_3_joint']}</param>
+          </state_interface>
+          <state_interface name="velocity"/>
+          <state_interface name="effort"/>
+        </joint>
+        <!-- NOTE:
+             Do NOT include ur_sensors / gpio blocks here
+             because MuJoCo hardware doesn't export those interfaces.
+        -->
+      </xacro:if>
+      <!-- ========================================================= -->
+      <!-- B) Real UR driver mode (use_mock_hardware:=false) -->
+      <!-- ========================================================= -->
+      <xacro:unless value="${use_mock_hardware}">
+        <hardware>
           <plugin>ur_robot_driver/URPositionHardwareInterface</plugin>
           <param name="robot_ip">${robot_ip}</param>
@@ -78,28 +140,240 @@
           <param name="tool_tcp_port">${tool_tcp_port}</param>
           <param name="robot_receive_timeout">${robot_receive_timeout}</param>
-        </xacro:unless>
-      </hardware>
-      <xacro:ur_joint_control_description
-        tf_prefix="${tf_prefix}"
-        initial_positions="${initial_positions}"
-      />
-      <!-- <xacro:ur_sensors
-        tf_prefix="${tf_prefix}"
-      /> -->
-      <!-- NOTE The following are joints used only for testing with mock hardware and will change in the future -->
-      <!-- <gpio name="${tf_prefix}speed_scaling">
-        <state_interface name="speed_scaling_factor">
-          <param name="initial_value">1.0</param>
-        </state_interface>
-        <command_interface name="target_speed_fraction_cmd"/>
-        <command_interface name="target_speed_fraction_async_success"/>
-      </gpio> -->
-      <!-- (rest of gpio and other definitions unchanged) -->
-      <!-- <gpio name="${tf_prefix}gpio"> -->
-        <!-- ... (same content as before) -->
-        <!-- <command_interface name="standard_digital_output_cmd_0"/> -->
-        <!-- truncated in this snippet for brevity, file should keep the full content -->
-      <!-- </gpio> -->
-      <!-- ... all other gpio blocks and definitions remain unchanged ... -->
+        </hardware>
+        <!-- Keep the original UR joint interface declaration (pos/vel/eff cmd + pos/vel/eff state) -->
+        <xacro:ur_joint_control_description
+          tf_prefix="${tf_prefix}"
+          initial_positions="${initial_positions}"
+        />
+        <!-- Keep UR sensors -->
+        <xacro:ur_sensors tf_prefix="${tf_prefix}" />
+        <!-- Keep the UR driver "mock/test" GPIO blocks exactly as before -->
+        <gpio name="${tf_prefix}speed_scaling">
+          <state_interface name="speed_scaling_factor">
+            <param name="initial_value">1.0</param>
+          </state_interface>
+          <command_interface name="target_speed_fraction_cmd"/>
+          <command_interface name="target_speed_fraction_async_success"/>
+        </gpio>
+        <gpio name="${tf_prefix}gpio">
+          <command_interface name="standard_digital_output_cmd_0"/>
+          <command_interface name="standard_digital_output_cmd_1"/>
+          <command_interface name="standard_digital_output_cmd_2"/>
+          <command_interface name="standard_digital_output_cmd_3"/>
+          <command_interface name="standard_digital_output_cmd_4"/>
+          <command_interface name="standard_digital_output_cmd_5"/>
+          <command_interface name="standard_digital_output_cmd_6"/>
+          <command_interface name="standard_digital_output_cmd_7"/>
+          <command_interface name="standard_digital_output_cmd_8"/>
+          <command_interface name="standard_digital_output_cmd_9"/>
+          <command_interface name="standard_digital_output_cmd_10"/>
+          <command_interface name="standard_digital_output_cmd_11"/>
+          <command_interface name="standard_digital_output_cmd_12"/>
+          <command_interface name="standard_digital_output_cmd_13"/>
+          <command_interface name="standard_digital_output_cmd_14"/>
+          <command_interface name="standard_digital_output_cmd_15"/>
+          <command_interface name="standard_digital_output_cmd_16"/>
+          <command_interface name="standard_digital_output_cmd_17"/>
+          <command_interface name="standard_analog_output_cmd_0"/>
+          <command_interface name="standard_analog_output_cmd_1"/>
+          <command_interface name="analog_output_domain_cmd"/>
+          <command_interface name="tool_voltage_cmd"/>
+          <command_interface name="io_async_success"/>
+          <state_interface name="digital_output_0"/>
+          <state_interface name="digital_output_1"/>
+          <state_interface name="digital_output_2"/>
+          <state_interface name="digital_output_3"/>
+          <state_interface name="digital_output_4"/>
+          <state_interface name="digital_output_5"/>
+          <state_interface name="digital_output_6"/>
+          <state_interface name="digital_output_7"/>
+          <state_interface name="digital_output_8"/>
+          <state_interface name="digital_output_9"/>
+          <state_interface name="digital_output_10"/>
+          <state_interface name="digital_output_11"/>
+          <state_interface name="digital_output_12"/>
+          <state_interface name="digital_output_13"/>
+          <state_interface name="digital_output_14"/>
+          <state_interface name="digital_output_15"/>
+          <state_interface name="digital_output_16"/>
+          <state_interface name="digital_output_17"/>
+          <state_interface name="digital_input_0"/>
+          <state_interface name="digital_input_1"/>
+          <state_interface name="digital_input_2"/>
+          <state_interface name="digital_input_3"/>
+          <state_interface name="digital_input_4"/>
+          <state_interface name="digital_input_5"/>
+          <state_interface name="digital_input_6"/>
+          <state_interface name="digital_input_7"/>
+          <state_interface name="digital_input_8"/>
+          <state_interface name="digital_input_9"/>
+          <state_interface name="digital_input_10"/>
+          <state_interface name="digital_input_11"/>
+          <state_interface name="digital_input_12"/>
+          <state_interface name="digital_input_13"/>
+          <state_interface name="digital_input_14"/>
+          <state_interface name="digital_input_15"/>
+          <state_interface name="digital_input_16"/>
+          <state_interface name="digital_input_17"/>
+          <state_interface name="standard_analog_output_0"/>
+          <state_interface name="standard_analog_output_1"/>
+          <state_interface name="standard_analog_input_0"/>
+          <state_interface name="standard_analog_input_1"/>
+          <state_interface name="analog_io_type_0"/>
+          <state_interface name="analog_io_type_1"/>
+          <state_interface name="analog_io_type_2"/>
+          <state_interface name="analog_io_type_3"/>
+          <state_interface name="tool_mode"/>
+          <state_interface name="tool_output_voltage"/>
+          <state_interface name="tool_output_current"/>
+          <state_interface name="tool_temperature"/>
+          <state_interface name="tool_analog_input_0"/>
+          <state_interface name="tool_analog_input_1"/>
+          <state_interface name="tool_analog_input_type_0"/>
+          <state_interface name="tool_analog_input_type_1"/>
+          <state_interface name="robot_mode"/>
+          <state_interface name="robot_status_bit_0"/>
+          <state_interface name="robot_status_bit_1"/>
+          <state_interface name="robot_status_bit_2"/>
+          <state_interface name="robot_status_bit_3"/>
+          <state_interface name="safety_mode"/>
+          <state_interface name="safety_status_bit_0"/>
+          <state_interface name="safety_status_bit_1"/>
+          <state_interface name="safety_status_bit_2"/>
+          <state_interface name="safety_status_bit_3"/>
+          <state_interface name="safety_status_bit_4"/>
+          <state_interface name="safety_status_bit_5"/>
+          <state_interface name="safety_status_bit_6"/>
+          <state_interface name="safety_status_bit_7"/>
+          <state_interface name="safety_status_bit_8"/>
+          <state_interface name="safety_status_bit_9"/>
+          <state_interface name="safety_status_bit_10"/>
+          <state_interface name="program_running"/>
+        </gpio>
+        <gpio name="${tf_prefix}payload">
+          <command_interface name="mass"/>
+          <command_interface name="cog.x"/>
+          <command_interface name="cog.y"/>
+          <command_interface name="cog.z"/>
+          <command_interface name="payload_async_success"/>
+        </gpio>
+        <gpio name="${tf_prefix}resend_robot_program">
+          <command_interface name="resend_robot_program_cmd"/>
+          <command_interface name="resend_robot_program_async_success"/>
+        </gpio>
+        <gpio name="${tf_prefix}hand_back_control">
+          <command_interface name="hand_back_control_cmd"/>
+          <command_interface name="hand_back_control_async_success"/>
+        </gpio>
+        <gpio name="${tf_prefix}zero_ftsensor">
+          <command_interface name="zero_ftsensor_cmd"/>
+          <command_interface name="zero_ftsensor_async_success"/>
+        </gpio>
+        <gpio name="${tf_prefix}freedrive_mode">
+          <command_interface name="async_success"/>
+          <command_interface name="enable"/>
+          <command_interface name="abort"/>
+        </gpio>
+        <gpio name="${tf_prefix}tool_contact">
+          <command_interface name="tool_contact_set_state"/>
+          <state_interface name="tool_contact_result"/>
+          <state_interface name="tool_contact_state"/>
+        </gpio>
+        <gpio name="${tf_prefix}system_interface">
+          <state_interface name="initialized"/>
+        </gpio>
+        <gpio name="${tf_prefix}force_mode">
+          <command_interface name="task_frame_x"/>
+          <command_interface name="task_frame_y"/>
+          <command_interface name="task_frame_z"/>
+          <command_interface name="task_frame_rx"/>
+          <command_interface name="task_frame_ry"/>
+          <command_interface name="task_frame_rz"/>
+          <command_interface name="selection_vector_x"/>
+          <command_interface name="selection_vector_y"/>
+          <command_interface name="selection_vector_z"/>
+          <command_interface name="selection_vector_rx"/>
+          <command_interface name="selection_vector_ry"/>
+          <command_interface name="selection_vector_rz"/>
+          <command_interface name="wrench_x"/>
+          <command_interface name="wrench_y"/>
+          <command_interface name="wrench_z"/>
+          <command_interface name="wrench_rx"/>
+          <command_interface name="wrench_ry"/>
+          <command_interface name="wrench_rz"/>
+          <command_interface name="limits_x"/>
+          <command_interface name="limits_y"/>
+          <command_interface name="limits_z"/>
+          <command_interface name="limits_rx"/>
+          <command_interface name="limits_ry"/>
+          <command_interface name="limits_rz"/>
+          <command_interface name="type"/>
+          <command_interface name="damping"/>
+          <command_interface name="gain_scaling"/>
+          <command_interface name="disable_cmd"/>
+          <command_interface name="force_mode_async_success"/>
+        </gpio>
+        <gpio name="${tf_prefix}trajectory_passthrough">
+          <command_interface name="setpoint_positions_0"/>
+          <command_interface name="setpoint_positions_1"/>
+          <command_interface name="setpoint_positions_2"/>
+          <command_interface name="setpoint_positions_3"/>
+          <command_interface name="setpoint_positions_4"/>
+          <command_interface name="setpoint_positions_5"/>
+          <command_interface name="setpoint_velocities_0"/>
+          <command_interface name="setpoint_velocities_1"/>
+          <command_interface name="setpoint_velocities_2"/>
+          <command_interface name="setpoint_velocities_3"/>
+          <command_interface name="setpoint_velocities_4"/>
+          <command_interface name="setpoint_velocities_5"/>
+          <command_interface name="setpoint_accelerations_0"/>
+          <command_interface name="setpoint_accelerations_1"/>
+          <command_interface name="setpoint_accelerations_2"/>
+          <command_interface name="setpoint_accelerations_3"/>
+          <command_interface name="setpoint_accelerations_4"/>
+          <command_interface name="setpoint_accelerations_5"/>
+          <command_interface name="transfer_state"/>
+          <command_interface name="time_from_start"/>
+          <command_interface name="abort"/>
+          <command_interface name="trajectory_size"/>
+        </gpio>
+        <gpio name="${tf_prefix}get_robot_software_version">
+          <state_interface name="get_version_major">
+            <param name="initial_value">1</param>
+          </state_interface>
+          <state_interface name="get_version_minor"/>
+          <state_interface name="get_version_build"/>
+          <state_interface name="get_version_bugfix"/>
+        </gpio>
+        <gpio name="${tf_prefix}motion_primitive">
+          <command_interface name="motion_type"/>
+          <command_interface name="q1"/>
+          <command_interface name="q2"/>
+          <command_interface name="q3"/>
+          <command_interface name="q4"/>
+          <command_interface name="q5"/>
+          <command_interface name="q6"/>
+          <command_interface name="pos_x"/>
+          <command_interface name="pos_y"/>
+          <command_interface name="pos_z"/>
+          <command_interface name="pos_qx"/>
+          <command_interface name="pos_qy"/>
+          <command_interface name="pos_qz"/>
+          <command_interface name="pos_qw"/>
+          <command_interface name="pos_via_x"/>
+          <command_interface name="pos_via_y"/>
+          <command_interface name="pos_via_z"/>
+          <command_interface name="pos_via_qx"/>
+          <command_interface name="pos_via_qy"/>
+          <command_interface name="pos_via_qz"/>
+          <command_interface name="pos_via_qw"/>
+          <command_interface name="blend_radius"/>
+          <command_interface name="velocity"/>
+          <command_interface name="acceleration"/>
+          <command_interface name="move_time"/>
+          <state_interface name="execution_status"/>
+          <state_interface name="ready_for_new_primitive"/>
+        </gpio>
+      </xacro:unless>
     </ros2_control>
   </xacro:macro>
